Commit message: Added in wheels and caster wheels to barista bot

File: barista_robot_description/urdf/barista_robot_model.urdf (robot description, URDF)
Before this commit: robot barista_bot, 2 links, 1 joints
Links:
- added link front_pitch_link, mass 0.010; collision sphere radius=0.0352; visual sphere radius=0.0352
- added link front_roll_link, mass 0.001; collision cylinder length=0.001 radius=0.0045000000000000005; visual cylinder length=0.001 radius=0.0045000000000000005
- added link front_yaw_link, mass 0.001; collision cylinder length=0.001 radius=0.0045000000000000005; visual cylinder length=0.001 radius=0.0045000000000000005
- added link left_wheel, mass 0.05; collision cylinder length=0.0206 radius=0.0352; visual cylinder length=0.0206 radius=0.0352
- added link rear_pitch_link, mass 0.010; collision sphere radius=0.0352; visual sphere radius=0.0352
- added link rear_roll_link, mass 0.001; collision cylinder length=0.001 radius=0.0045000000000000005; visual cylinder length=0.001 radius=0.0045000000000000005
- added link rear_yaw_link, mass 0.001; collision cylinder length=0.001 radius=0.0045000000000000005; visual cylinder length=0.001 radius=0.0045000000000000005
- added link right_wheel, mass 0.05; collision cylinder length=0.0206 radius=0.0352; visual cylinder length=0.0206 radius=0.0352
Joints:
- added joint front_pitch_joint: type continuous, parent front_roll_link, child front_pitch_link, origin xyz=0 0 0 rpy=0 0 0, axis 0 1 0, limit effort=1000.0 velocity=100.0
- added joint front_roll_joint: type continuous, parent front_yaw_link, child front_roll_link, origin xyz=0 0 0 rpy=0 0 0, axis 1 0 0, limit effort=1000.0 velocity=100.0
- added joint front_yaw_joint: type continuous, parent main_body, child front_yaw_link, origin xyz=0 0.138 -0.0775 rpy=0 0 0, axis 0 0 1, limit effort=1000.0 velocity=100.0
- added joint joint_left_wheel: type continuous, parent main_body, child left_wheel, origin xyz=0.158 0 -0.0775 rpy=0 0 0, axis 1 0 0, limit effort=10000 velocity=1000
- added joint joint_right_wheel: type continuous, parent main_body, child right_wheel, origin xyz=-0.158 0 -0.0775 rpy=0 0 0, axis 1 0 0, limit effort=10000 velocity=1000
- added joint rear_pitch_joint: type continuous, parent rear_roll_link, child rear_pitch_link, origin xyz=0 0 0 rpy=0 0 0, axis 0 1 0, limit effort=1000.0 velocity=100.0
- added joint rear_roll_joint: type continuous, parent rear_yaw_link, child rear_roll_link, origin xyz=0 0 0 rpy=0 0 0, axis 1 0 0, limit effort=1000.0 velocity=100.0
- added joint rear_yaw_joint: type continuous, parent main_body, child rear_yaw_link, origin xyz=0 -0.138 -0.0775 rpy=0 0 0, axis 0 0 1, limit effort=1000.0 velocity=100.0

Commit message: Added in differential drive and fixed wheel orientation to match ROS standard.

File: barista_robot_description/urdf/barista_robot_model.urdf (robot description, URDF)
Before this commit: robot barista_bot, 10 links, 9 joints
Joints:
- joint front_yaw_joint: origin xyz=0 0.138 -0.0775 rpy=0 0 0 -> xyz=0.138 0 -0.0775 rpy=0 0 0
- joint joint_left_wheel: axis 1 0 0 -> 0 1 0; origin xyz=0.158 0 -0.0775 rpy=0 0 0 -> xyz=0 0.158 -0.0775 rpy=0 0 0
- joint joint_right_wheel: axis 1 0 0 -> 0 1 0; origin xyz=-0.158 0 -0.0775 rpy=0 0 0 -> xyz=0 -0.158 -0.0775 rpy=0 0 0
- joint rear_yaw_joint: origin xyz=0 -0.138 -0.0775 rpy=0 0 0 -> xyz=-0.138 0 -0.0775 rpy=0 0 0

Commit message: Added in lidar sensor to barista bot, modified world to include obstacle

File: barista_robot_description/urdf/barista_robot_model.urdf (robot description, URDF)
Before this commit: robot barista_bot, 10 links, 9 joints
Links:
- added link cupholder_tray_link, mass 0.2; collision cylinder length=0.090 radius=0.160; visual cylinder length=0.090 radius=0.160
- added link laser_scan_frame
- added link laser_scan_link, mass 0.1; collision box size=0.01 0.01 0.01; visual mesh filename=package://barista_robot_description/meshes/velodyne_puck.dae scale=1 1 1
- added link standoff_rod_1_link, mass 0.05; collision cylinder length=0.220 radius=0.01; visual cylinder length=0.220 radius=0.01
- added link standoff_rod_2_link, mass 0.05; collision cylinder length=0.220 radius=0.01; visual cylinder length=0.220 radius=0.01
- added link standoff_rod_3_link, mass 0.05; collision cylinder length=0.220 radius=0.01; visual cylinder length=0.220 radius=0.01
- added link standoff_rod_4_link, mass 0.05; collision cylinder length=0.220 radius=0.01; visual cylinder length=0.220 radius=0.01
Joints:
- added joint cupholder_tray_link_joint: type fixed, parent main_body, child cupholder_tray_link, origin xyz=0 0 0.3425 rpy=0 0 0
- added joint laser_scan_frame_joint: type fixed, parent laser_scan_link, child laser_scan_frame, origin xyz=0 0 0.04 rpy=0 0 0, axis 0 0 0
- added joint laser_scan_joint: type fixed, parent main_body, child laser_scan_link, origin xyz=0.118 0 0.0775 rpy=0 0 0
- added joint standoff_rod_1_joint: type fixed, parent main_body, child standoff_rod_1_link, origin xyz=0.06 0.128 0.1875 rpy=0 0 0
- added joint standoff_rod_2_joint: type fixed, parent main_body, child standoff_rod_2_link, origin xyz=-0.06 0.128 0.1875 rpy=0 0 0
- added joint standoff_rod_3_joint: type fixed, parent main_body, child standoff_rod_3_link, origin xyz=0.06 -0.128 0.1875 rpy=0 0 0
- added joint standoff_rod_4_joint: type fixed, parent main_body, child standoff_rod_4_link, origin xyz=-0.06 -0.128 0.1875 rpy=0 0 0
