Commit message: Added in driver and caster wheel xacro to barista robot and differential drive capabilities

File: barista_robot_description/xacro/barista_robot_model.urdf.xacro (robot description, xacro)
@@ -2,13 +2,27 @@
 <robot xmlns:xacro="http://www.ros.org/wiki/xacro" name="barista_bot">
   <xacro:include filename="$(find barista_robot_description)/xacro/inertia_calculations.xacro"/>
-  <!-- <xacro:include filename="$(find barista_robot_description)/xacro/drive_wheel.xacro" /> -->
+  <xacro:include filename="$(find barista_robot_description)/xacro/drive_wheel.xacro" />
+  <xacro:include filename="$(find barista_robot_description)/xacro/caster_wheel.xacro" />
   <xacro:property name="body_radius" value="0.178"/>
   <xacro:property name="body_height" value="0.155"/>
-  <xacro:property name="body_height" value="0.1"/>
   <xacro:property name="body_mass" value="0.5"/>
-  <xacro:property name="wheel_width" value="0.001"/>
-  <xacro:property name="wheel_radius" value="0.035"/>
+  <xacro:property name="wheel_width" value="0.0206"/>
+  <xacro:property name="wheel_radius" value="0.0352"/>
+  <xacro:property name="wheel_mass" value="0.05"/>
+  <xacro:property name="wheel_rpy" value="1.5707 1.5707 0"/>
   <material name="blue">
       <color rgba="0.0 0.0 1.0 1"/>
+  </material>
+  <material name="yellow">
+      <color rgba="1.0 1.0 0.0 1"/>
+  </material>
+  <material name="red">
+      <color rgba="1.0 0.0 0.0 1"/>
+  </material>
+  <material name="green_dark">
+    <color rgba="0.0 0.5 0.0 1"/>
+  </material>
+  <material name="black">
+      <color rgba="0.0 0.0 0.0 1"/>
   </material>
   <link name="base_link">
@@ -37,3 +51,84 @@
     <child link="main_body" />
   </joint>
+  <!-- Left Wheel -->
+  <xacro:wheel_macro
+      wheel_name="left_wheel"
+      radius="${wheel_radius}"
+      length="${wheel_width}"
+      mass="${wheel_mass}"
+      rpy="${wheel_rpy}"/>
+  <joint name="joint_left_wheel" type="continuous">
+    <origin rpy="0 0 0" xyz="0 0.158 -0.0775"/>
+    <child link="left_wheel"/>
+    <parent link="main_body"/>
+    <axis rpy="0 0 0" xyz="0 1 0"/>
+    <limit effort="10000" velocity="1000"/>
+    <joint_properties damping="1.0" friction="1.0"/>
+  </joint>
+  <!-- Right Wheel -->
+  <xacro:wheel_macro
+      wheel_name="right_wheel"
+      radius="${wheel_radius}"
+      length="${wheel_width}"
+      mass="${wheel_mass}"
+      rpy="${wheel_rpy}"/>
+  <joint name="joint_right_wheel" type="continuous">
+    <origin rpy="0 0 0" xyz="0 -0.158 -0.0775"/>
+    <child link="right_wheel"/>
+    <parent link="main_body"/>
+    <axis rpy="0 0 0" xyz="0 1 0"/>
+    <limit effort="10000" velocity="1000"/>
+    <joint_properties damping="1.0" friction="1.0"/>
+  </joint>
+  <!-- Front Caster Wheel -->
+  <xacro:caster_wheel_macro
+      caster_wheel_name="front"
+      radius="${wheel_radius}"
+      caster_color="red"/>
+    <joint name="front_yaw_joint" type="continuous">
+        <origin rpy="0 0 0" xyz="0.138 0 -0.0775" />
+        <parent link="main_body" />
+        <child link="front_yaw_link" />
+        <axis xyz="0 0 1" />
+        <limit effort="1000.0" velocity="100.0" />
+        <dynamics damping="0.0" friction="0.1"/>
+    </joint>
+  <!-- Rear Caster Wheel -->
+  <xacro:caster_wheel_macro
+      caster_wheel_name="rear"
+      radius="${wheel_radius}"
+      caster_color="green_dark"/>
+  <joint name="rear_yaw_joint" type="continuous">
+    <origin rpy="0 0 0" xyz="-0.138 0 -0.0775" />
+    <parent link="main_body" />
+    <child link="rear_yaw_link" />
+    <axis xyz="0 0 1" />
+    <limit effort="1000.0" velocity="100.0" />
+    <dynamics damping="0.0" friction="0.1"/>
+  </joint>
+  <!-- Differential Drive Plugin -->
+  <gazebo>
+    <plugin
+        filename="gz-sim-diff-drive-system"
+        name="gz::sim::systems::DiffDrive">
+        <left_joint>joint_left_wheel</left_joint>
+        <right_joint>joint_right_wheel</right_joint>
+        <wheel_separation>0.316</wheel_separation>
+        <wheel_radius>0.0352</wheel_radius>
+        <topic>cmd_vel</topic>
+        <publish_odom>true</publish_odom>
+        <publish_odom_tf>true</publish_odom_tf>
+        <publish_wheel_tf>true</publish_wheel_tf>
+        <odom_topic>odom</odom_topic>
+        <tf_topic>tf</tf_topic>
+        <frame_id>odom</frame_id>
+        <child_frame_id>base_link</child_frame_id>
+    </plugin>
+  </gazebo>
+  <!-- Joint state publisher plugin -->
+  <gazebo>
+    <plugin filename="gz-sim-joint-state-publisher-system"
+          name="gz::sim::systems::JointStatePublisher">
+    </plugin>
+  </gazebo>
 </robot>

File: barista_robot_description/xacro/inertia_calculations.xacro (robot description, xacro)
@@ -1,16 +1,31 @@
 <?xml version="1.0"?>
 <robot xmlns:xacro="http://www.ros.org/wiki/xacro">
-  <xacro:macro name="cylinder_inertia" params="mass radius length">
-    <inertial>
-      <mass value="${mass}"/>
-      <origin rpy="0 0 0" xyz="0 0 0"/>
-      <inertia
-        ixx="${mass * (3*radius*radius + length*length) / 12.0}"
-        ixy="0.0"
-        ixz="0.0"
-        iyy="${mass * (3*radius*radius + length*length) / 12.0}"
-        iyz="0.0"
-        izz="${0.5 * mass * radius * radius}" />
-    </inertial>
-  </xacro:macro>
+<xacro:macro name="cylinder_inertia"
+             params="mass radius length xyz:='0 0 0' rpy:='0 0 0'">
+  <inertial>
+    <origin xyz="${xyz}" rpy="${rpy}"/>
+    <mass value="${mass}"/>
+    <inertia
+      ixx="${mass * (3*radius*radius + length*length) / 12.0}"
+      ixy="0.0"
+      ixz="0.0"
+      iyy="${mass * (3*radius*radius + length*length) / 12.0}"
+      iyz="0.0"
+      izz="${0.5 * mass * radius * radius}"/>
+  </inertial>
+</xacro:macro>
+<xacro:macro name="sphere_inertia"
+             params="mass radius xyz:='0 0 0' rpy:='0 0 0'">
+  <inertial>
+    <origin xyz="${xyz}" rpy="${rpy}"/>
+    <mass value="${mass}"/>
+    <inertia
+      ixx="${mass * (2*radius*radius ) / 5.0}"
+      ixy="0.0"
+      ixz="0.0"
+      iyy="${mass * (2*radius*radius ) / 5.0}"
+      iyz="0.0"
+      izz="${mass * (2*radius*radius ) / 5.0}"/>
+  </inertial>
+</xacro:macro>
 </robot>

Commit message: Modified caster and drive wheels to be more modular

File: barista_robot_description/xacro/barista_robot_model.urdf.xacro (robot description, xacro)
@@ -57,6 +57,8 @@
       length="${wheel_width}"
       mass="${wheel_mass}"
-      rpy="${wheel_rpy}"/>
-  <joint name="joint_left_wheel" type="continuous">
+      rpy="${wheel_rpy}"
+      parent_link="main_body"
+      joint_xyz="0 0.158 -0.0775"/>
+  <!-- <joint name="joint_left_wheel" type="continuous">
     <origin rpy="0 0 0" xyz="0 0.158 -0.0775"/>
     <child link="left_wheel"/>
@@ -65,5 +67,5 @@
     <limit effort="10000" velocity="1000"/>
     <joint_properties damping="1.0" friction="1.0"/>
-  </joint>
+  </joint> -->
   <!-- Right Wheel -->
   <xacro:wheel_macro
@@ -72,6 +74,8 @@
       length="${wheel_width}"
       mass="${wheel_mass}"
-      rpy="${wheel_rpy}"/>
-  <joint name="joint_right_wheel" type="continuous">
+      rpy="${wheel_rpy}"
+      parent_link="main_body"
+      joint_xyz="0 -0.158 -0.0775"/>
+  <!-- <joint name="joint_right_wheel" type="continuous">
     <origin rpy="0 0 0" xyz="0 -0.158 -0.0775"/>
     <child link="right_wheel"/>
@@ -80,11 +84,13 @@
     <limit effort="10000" velocity="1000"/>
     <joint_properties damping="1.0" friction="1.0"/>
-  </joint>
+  </joint> -->
   <!-- Front Caster Wheel -->
   <xacro:caster_wheel_macro
       caster_wheel_name="front"
       radius="${wheel_radius}"
-      caster_color="red"/>
-    <joint name="front_yaw_joint" type="continuous">
+      caster_color="red"
+      parent_link="main_body"
+      joint_xyz="0.138 0 -0.0775"/>
+    <!-- <joint name="front_yaw_joint" type="continuous">
         <origin rpy="0 0 0" xyz="0.138 0 -0.0775" />
         <parent link="main_body" />
@@ -93,11 +99,13 @@
         <limit effort="1000.0" velocity="100.0" />
         <dynamics damping="0.0" friction="0.1"/>
-    </joint>
+    </joint> -->
   <!-- Rear Caster Wheel -->
   <xacro:caster_wheel_macro
       caster_wheel_name="rear"
       radius="${wheel_radius}"
-      caster_color="green_dark"/>
-  <joint name="rear_yaw_joint" type="continuous">
+      caster_color="green_dark"
+      parent_link="main_body"
+      joint_xyz="-0.138 0 -0.0775"/>
+  <!-- <joint name="rear_yaw_joint" type="continuous">
     <origin rpy="0 0 0" xyz="-0.138 0 -0.0775" />
     <parent link="main_body" />
@@ -106,5 +114,5 @@
     <limit effort="1000.0" velocity="100.0" />
     <dynamics damping="0.0" friction="0.1"/>
-  </joint>
+  </joint> -->
   <!-- Differential Drive Plugin -->
   <gazebo>

File: barista_robot_description/xacro/caster_wheel.xacro (robot description, xacro)
@@ -2,5 +2,5 @@
 <robot xmlns:xacro="http://www.ros.org/wiki/xacro">
   <xacro:include filename="$(find barista_robot_description)/xacro/inertia_calculations.xacro"/>
-  <xacro:macro name="caster_wheel_macro" params="caster_wheel_name radius caster_color">
+  <xacro:macro name="caster_wheel_macro" params="caster_wheel_name parent_link joint_xyz radius caster_color">
     <link name="${caster_wheel_name}_yaw_link">
         <visual>
@@ -23,4 +23,12 @@
         rpy="0 1.5707 1.5707"/>
     </link>
+    <joint name="${caster_wheel_name}_yaw_joint" type="continuous">
+        <origin rpy="0 0 0" xyz="${joint_xyz}" />
+        <parent link="${parent_link}" />
+        <child link="${caster_wheel_name}_yaw_link" />
+        <axis xyz="0 0 1" />
+        <limit effort="1000.0" velocity="100.0" />
+        <dynamics damping="0.0" friction="0.1"/>
+    </joint>
     <link name="${caster_wheel_name}_roll_link">
         <visual>

File: barista_robot_description/xacro/drive_wheel.xacro (robot description, xacro)
@@ -2,5 +2,5 @@
 <robot xmlns:xacro="http://www.ros.org/wiki/xacro">
   <xacro:include filename="$(find barista_robot_description)/xacro/inertia_calculations.xacro"/>
-  <xacro:macro name="wheel_macro" params="wheel_name radius length mass xyz:='0 0 0' rpy:='0 0 0'">
+  <xacro:macro name="wheel_macro" params="wheel_name parent_link joint_xyz radius length mass xyz:='0 0 0' rpy:='0 0 0'">
     <link name="${wheel_name}">
         <visual>
@@ -22,4 +22,12 @@
       length="${length}"/>
     </link>
+  <joint name="joint_${wheel_name}" type="continuous">
+    <origin rpy="0 0 0" xyz="${joint_xyz}"/>
+    <child link="${wheel_name}"/>
+    <parent link="${parent_link}"/>
+    <axis rpy="0 0 0" xyz="0 1 0"/>
+    <limit effort="10000" velocity="1000"/>
+    <joint_properties damping="1.0" friction="1.0"/>
+  </joint>
     <gazebo reference="${wheel_name}">
         <collision>

Commit message: Added in cupholder tray and standoff rods

File: barista_robot_description/xacro/barista_robot_model.urdf.xacro (robot description, xacro)
@@ -4,4 +4,6 @@
   <xacro:include filename="$(find barista_robot_description)/xacro/drive_wheel.xacro" />
   <xacro:include filename="$(find barista_robot_description)/xacro/caster_wheel.xacro" />
+  <xacro:include filename="$(find barista_robot_description)/xacro/standoff_rod.xacro" />
+  <xacro:include filename="$(find barista_robot_description)/xacro/cup_holder_tray.xacro" />
   <xacro:property name="body_radius" value="0.178"/>
   <xacro:property name="body_height" value="0.155"/>
@@ -11,4 +13,10 @@
   <xacro:property name="wheel_mass" value="0.05"/>
   <xacro:property name="wheel_rpy" value="1.5707 1.5707 0"/>
+  <xacro:property name="standoff_rod_length" value="0.220"/>
+  <xacro:property name="standoff_rod_radius" value="0.01"/>
+  <xacro:property name="standoff_rod_mass" value="0.05"/>
+  <xacro:property name="cupholder_tray_length" value="0.090"/>
+  <xacro:property name="cupholder_tray_radius" value="0.160"/>
+  <xacro:property name="cupholder_tray_mass" value="0.2"/>
   <material name="blue">
       <color rgba="0.0 0.0 1.0 1"/>
@@ -25,4 +33,7 @@
   <material name="black">
       <color rgba="0.0 0.0 0.0 1"/>
+  </material>
+  <material name="grey">
+      <color rgba="0.5 0.5 0.5 1"/>
   </material>
   <link name="base_link">
@@ -60,12 +71,4 @@
       parent_link="main_body"
       joint_xyz="0 0.158 -0.0775"/>
-  <!-- <joint name="joint_left_wheel" type="continuous">
-    <origin rpy="0 0 0" xyz="0 0.158 -0.0775"/>
-    <child link="left_wheel"/>
-    <parent link="main_body"/>
-    <axis rpy="0 0 0" xyz="0 1 0"/>
-    <limit effort="10000" velocity="1000"/>
-    <joint_properties damping="1.0" friction="1.0"/>
-  </joint> -->
   <!-- Right Wheel -->
   <xacro:wheel_macro
@@ -77,12 +80,4 @@
       parent_link="main_body"
       joint_xyz="0 -0.158 -0.0775"/>
-  <!-- <joint name="joint_right_wheel" type="continuous">
-    <origin rpy="0 0 0" xyz="0 -0.158 -0.0775"/>
-    <child link="right_wheel"/>
-    <parent link="main_body"/>
-    <axis rpy="0 0 0" xyz="0 1 0"/>
-    <limit effort="10000" velocity="1000"/>
-    <joint_properties damping="1.0" friction="1.0"/>
-  </joint> -->
   <!-- Front Caster Wheel -->
   <xacro:caster_wheel_macro
@@ -92,12 +87,4 @@
       parent_link="main_body"
       joint_xyz="0.138 0 -0.0775"/>
-    <!-- <joint name="front_yaw_joint" type="continuous">
-        <origin rpy="0 0 0" xyz="0.138 0 -0.0775" />
-        <parent link="main_body" />
-        <child link="front_yaw_link" />
-        <axis xyz="0 0 1" />
-        <limit effort="1000.0" velocity="100.0" />
-        <dynamics damping="0.0" friction="0.1"/>
-    </joint> -->
   <!-- Rear Caster Wheel -->
   <xacro:caster_wheel_macro
@@ -107,12 +94,43 @@
       parent_link="main_body"
       joint_xyz="-0.138 0 -0.0775"/>
-  <!-- <joint name="rear_yaw_joint" type="continuous">
-    <origin rpy="0 0 0" xyz="-0.138 0 -0.0775" />
-    <parent link="main_body" />
-    <child link="rear_yaw_link" />
-    <axis xyz="0 0 1" />
-    <limit effort="1000.0" velocity="100.0" />
-    <dynamics damping="0.0" friction="0.1"/>
-  </joint> -->
+  <!-- Standoff rod 1 -->
+  <xacro:standoff_rod_macro
+      standoff_rod_name="standoff_rod_1"
+      radius="${standoff_rod_radius}"
+      length="${standoff_rod_length}"
+      mass="${standoff_rod_mass}"
+      parent_link="main_body"
+      joint_xyz="0.06 0.128 0.1875"/>
+  <!-- Standoff rod 2 -->
+  <xacro:standoff_rod_macro
+      standoff_rod_name="standoff_rod_2"
+      radius="${standoff_rod_radius}"
+      length="${standoff_rod_length}"
+      mass="${standoff_rod_mass}"
+      parent_link="main_body"
+      joint_xyz="-0.06 0.128 0.1875"/>
+  <!-- Standoff rod 3 -->
+  <xacro:standoff_rod_macro
+      standoff_rod_name="standoff_rod_3"
+      radius="${standoff_rod_radius}"
+      length="${standoff_rod_length}"
+      mass="${standoff_rod_mass}"
+      parent_link="main_body"
+      joint_xyz="0.06 -0.128 0.1875"/>
+  <!-- Standoff rod 4 -->
+  <xacro:standoff_rod_macro
+      standoff_rod_name="standoff_rod_4"
+      radius="${standoff_rod_radius}"
+      length="${standoff_rod_length}"
+      mass="${standoff_rod_mass}"
+      parent_link="main_body"
+      joint_xyz="-0.06 -0.128 0.1875"/>
+  <!-- Cupholder tray -->
+  <xacro:cupholder_tray_macro
+      radius="${cupholder_tray_radius}"
+      length="${cupholder_tray_length}"
+      mass="${cupholder_tray_mass}"
+      parent_link="main_body"
+      joint_xyz="0 0 0.3425"/>
   <!-- Differential Drive Plugin -->
   <gazebo>

Commit message: Added in conditional laser scanner to barista robot

File: barista_robot_description/xacro/barista_robot_model.urdf.xacro (robot description, xacro)
@@ -1,4 +1,7 @@
 <?xml version="1.0"?>
 <robot xmlns:xacro="http://www.ros.org/wiki/xacro" name="barista_bot">
+  <!-- Laser scanner -->
+  <xacro:arg name="include_laser" default="true"/>
+  <xacro:property name="include_laser" value="$(arg include_laser)"/>
   <xacro:include filename="$(find barista_robot_description)/xacro/inertia_calculations.xacro"/>
   <xacro:include filename="$(find barista_robot_description)/xacro/drive_wheel.xacro" />
@@ -6,4 +9,5 @@
   <xacro:include filename="$(find barista_robot_description)/xacro/standoff_rod.xacro" />
   <xacro:include filename="$(find barista_robot_description)/xacro/cup_holder_tray.xacro" />
+  <xacro:include filename="$(find barista_robot_description)/xacro/laser_scanner.xacro" />
   <xacro:property name="body_radius" value="0.178"/>
   <xacro:property name="body_height" value="0.155"/>

Commit message: Modified xacro file to allow for robot model name and color, allowing for spawn of multiple robots

File: barista_robot_description/xacro/barista_robot_model.urdf.xacro (robot description, xacro)
@@ -1,7 +1,13 @@
 <?xml version="1.0"?>
-<robot xmlns:xacro="http://www.ros.org/wiki/xacro" name="barista_bot">
+<robot xmlns:xacro="http://www.ros.org/wiki/xacro" name="barista_robot">
   <!-- Laser scanner -->
   <xacro:arg name="include_laser" default="true"/>
   <xacro:property name="include_laser" value="$(arg include_laser)"/>
+  <!-- Robot color -->
+  <xacro:arg name="robot_color" default="blue"/>
+  <xacro:property name="robot_color" value="$(arg robot_color)"/>
+  <!-- Robot name -->
+  <xacro:arg name="robot_name" default="barista_bot"/>
+  <xacro:property name="robot_name" value="$(arg robot_name)"/>
   <xacro:include filename="$(find barista_robot_description)/xacro/inertia_calculations.xacro"/>
   <xacro:include filename="$(find barista_robot_description)/xacro/drive_wheel.xacro" />
@@ -49,5 +55,5 @@
         <cylinder length="${body_height}" radius="${body_radius}"/>
       </geometry>
-      <material name="blue"/>
+      <material name="${robot_color}"/>
     </visual>
     <collision>
@@ -93,5 +99,5 @@
   <!-- Rear Caster Wheel -->
   <xacro:caster_wheel_macro
-      caster_wheel_name="rear"
+      caster_wheel_name="back"
       radius="${wheel_radius}"
       caster_color="green_dark"
@@ -146,12 +152,12 @@
         <wheel_separation>0.316</wheel_separation>
         <wheel_radius>0.0352</wheel_radius>
-        <topic>cmd_vel</topic>
+        <topic>${robot_name}/cmd_vel</topic>
         <publish_odom>true</publish_odom>
         <publish_odom_tf>true</publish_odom_tf>
         <publish_wheel_tf>true</publish_wheel_tf>
-        <odom_topic>odom</odom_topic>
+        <odom_topic>${robot_name}/odom</odom_topic>
         <tf_topic>tf</tf_topic>
-        <frame_id>odom</frame_id>
-        <child_frame_id>base_link</child_frame_id>
+        <frame_id>${robot_name}/odom</frame_id>
+        <child_frame_id>${robot_name}/base_link</child_frame_id>
     </plugin>
   </gazebo>
@@ -159,6 +165,22 @@
   <gazebo>
     <plugin filename="gz-sim-joint-state-publisher-system"
+            name="gz::sim::systems::JointStatePublisher">
+        <topic>${robot_name}/joint_states</topic>
+        <update_rate>30</update_rate>
+        <!-- Publish the state of these joints -->
+        <joint_name>joint_left_wheel</joint_name>
+        <joint_name>joint_right_wheel</joint_name>
+        <joint_name>front_yaw_joint</joint_name>
+        <joint_name>back_yaw_joint</joint_name>
+        <joint_name>front_roll_joint</joint_name>
+        <joint_name>back_roll_joint</joint_name>
+        <joint_name>front_pitch_joint</joint_name>
+        <joint_name>back_pitch_joint</joint_name>
+    </plugin>
+  </gazebo>
+  <!-- <gazebo>
+    <plugin filename="gz-sim-joint-state-publisher-system"
           name="gz::sim::systems::JointStatePublisher">
     </plugin>
-  </gazebo>
+  </gazebo> -->
 </robot>

File: barista_robot_description/xacro/laser_scanner.xacro (robot description, xacro)
@@ -44,9 +44,9 @@
         <sensor type="gpu_lidar" name="gpu_lidar">
             <pose relative_to='laser_scan_frame'>0 0 0 0 0 0</pose>
-            <gz_frame_id>laser_scan_frame</gz_frame_id>
+            <gz_frame_id>${robot_name}/laser_scan_frame</gz_frame_id>
             <always_on>1</always_on>
             <visualize>true</visualize>
             <update_rate>100</update_rate>
-            <topic>laser_scan</topic>
+            <topic>${robot_name}/laser_scan</topic>
             <ray>
                 <scan>

Commit message: Added in two robot launch file for rick and morty bots

File: barista_robot_description/xacro/barista_robot_model.urdf.xacro (robot description, xacro)
@@ -142,5 +142,6 @@
       mass="${cupholder_tray_mass}"
       parent_link="main_body"
-      joint_xyz="0 0 0.3425"/>
+      joint_xyz="0 0 0.3425"
+      robot_color="${robot_color}"/>
   <!-- Differential Drive Plugin -->
   <gazebo>

File: barista_robot_description/xacro/cup_holder_tray.xacro (robot description, xacro)
@@ -2,5 +2,5 @@
 <robot xmlns:xacro="http://www.ros.org/wiki/xacro">
   <xacro:include filename="$(find barista_robot_description)/xacro/inertia_calculations.xacro"/>
-  <xacro:macro name="cupholder_tray_macro" params="parent_link joint_xyz length radius mass">
+  <xacro:macro name="cupholder_tray_macro" params="parent_link joint_xyz length radius mass robot_color">
     <link name="cupholder_tray_link">
     <visual>
@@ -8,5 +8,5 @@
         <cylinder length="${length}" radius="${radius}"/>
         </geometry>
-        <material name="blue"/>
+        <material name="${robot_color}"></material>
     </visual>
     <collision>

File: barista_robot_description/xacro/laser_scanner.xacro (robot description, xacro)
@@ -33,11 +33,11 @@
         <axis xyz="0 0 0"/>
     </joint>
-    <!-- Enable Sensors in Gazebo Sim -->
+    <!-- Enable Sensors in Gazebo Sim
     <gazebo>
         <plugin filename="gz-sim-sensors-system" name="gz::sim::systems::Sensors">
-            <!-- use ogre2 if ogre v2.x is installed, otherwise use ogre -->
+            use ogre2 if ogre v2.x is installed, otherwise use ogre
             <render_engine>ogre2</render_engine>
         </plugin>
-    </gazebo>
+    </gazebo> -->
     <!-- Laser Scanner Plugin -->
     <gazebo reference="laser_scan_frame">
